File: Bat Listener Hardware/Bat_Listener_v4_KiCAD/Bat_Listener_v4.sch (KiCad schematic (older format))
At the start: 57 parts, among them J1 PHONES, P1 ULTRASON, P10 LOGO1, P11 LOGO2, P12 Hex_Spacer, P13 FREQ_SELECT_1, P14 FREQ_SELECT_IN, P2 uP O/P, P3 NO_Pb, P4 BAT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

Commit message: Update of PCB and Enclosure Files
Added headphone socket.
Parts:
- D4: symbol Device:LED -> Bat_Listener_v4-rescue:LED-Device
Changed lines of the file:
@@
 VIRTUAL \nGROUND
 $Comp
-L Device:LED D4
+L Bat_Listener_v4-rescue:LED-Device D4
 U 1 1 57B2D840
 P 8650 4700
