File: Bat Listener Hardware/Bat_Listener_v4_KiCAD/Bat_Listener_v4.kicad_pcb (KiCad board)
At the start: 2 copper layers, 50 x 100 mm, 51 parts, among them J1 PHONES, P1 ULTRASON, P10 LOGO1, P11 LOGO2, P2 uP O/P, P3 NO_Pb, P4 BAT, P5 PCB, Q1 BC337, SW1 ON/OFF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

Commit message: updated instructions - small change
Other:
- net class Default removed
